File: Hardware/MachineLearning-MM-Carrier.brd (EAGLE design)
At the start: 58.4 x 52.1 mm, 138 parts, among them J11 microSD, J2 JTAG, J3 QWIIC_RIGHT_ANGLE, J4 MICROMOD-2222-C, J5 SPI, J6 UART, J7 CAMERA-HIMAXFACEUP, J8 Dedicated, U3 AP2127K-1.8V, U4 LIS2DH12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

Commit message: Rename SPI lines for clarification
Connections:
- net SPI_SDI renamed SPI_CIPO
- net SPI_SDO renamed SPI_COPI
Changed lines of the file:
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@@
 <layer number="47" name="Measures" color="7" fill="1" visible="no" active="yes"/>
 <layer number="48" name="Document" color="7" fill="1" visible="no" active="yes"/>
-<layer number="49" name="Reference" color="7" fill="1" visible="yes" active="yes"/>
+<layer number="49" name="Reference" color="7" fill="1" visible="no" active="yes"/>
 <layer number="50" name="dxf" color="7" fill="1" visible="no" active="yes"/>
 <layer number="51" name="tDocu" color="6" fill="1" visible="yes" active="yes"/>
@@
 </elements>
 <signals>
-<signal name="SPI_SDI">
+<signal name="SPI_CIPO">
 <contactref element="J11" pad="DO/DAT0"/>
 <wire x1="45.92" y1="44.99" x2="45.92" y2="43.234" width="0.1778" layer="1"/>
@@
 <wire x1="17.348" y1="25.07" x2="16.3999" y2="26.0181" width="0.1778" layer="1"/>
 </signal>
-<signal name="SPI_SDO">
+<signal name="SPI_COPI">
 <contactref element="J11" pad="DI/CMD"/>
 <wire x1="41.52" y1="44.99" x2="41.529" y2="44.981" width="0.1778" layer="1"/>
